File: PCB/LineSensor/LineBoard_pro/LineBoard_pro.kicad_pcb (KiCad board)
At the start: 2 copper layers, 20 parts, among them IC1 NJL7502R, IC2 NJL7502R, IC3 NJL7502R, IC4 NJL7502R, J1 to MAIN, U1 TMUX1204DGSR

Commit message: ラインセンサ完成
Parts:
- moved C1 5.32 mm to (96.9, 37.3)
- moved C2 4.10 mm to (102.6, 35.1), turned to -90 degrees
- moved J1 0.60 mm to (96.0, 40.6)
- moved U1 0.32 mm to (100.1, 33.7), turned to 90 degrees
Routing:
- net +3V3: track 0.00 -> 83.9 mm, vias 0 -> 6
- net GND: track 0.00 -> 71.8 mm, vias 0 -> 100
- net /S3: track 0.00 -> 28.1 mm, vias 0 -> 1
- net /S0: track 0.00 -> 25.1 mm, vias 0 -> 1
- net /S1: track 0.00 -> 19.0 mm, vias 0 -> 1
- net /S2: track 0.00 -> 13.4 mm, vias 0 -> 1
- net /Line_A1: track 0.00 -> 13.0 mm, vias 0 -> 1
- net /Line_OUT: track 0.00 -> 9.29 mm, vias 0 -> 1
- net /Line_A0: track 0.00 -> 6.20 mm
- net Net-(D4-A): vias 0 -> 1
- net Net-(D3-A): vias 0 -> 1
- net Net-(D2-A): vias 0 -> 1
- net Net-(D1-A): vias 0 -> 1
- added copper zone on B.Cu, net GND
- added copper zone on F.Cu, net GND
Other:
- board outline added: 60 x 15 mm

Commit message: ソレノイド基板作成開始
Routing:
- net GND: vias 100 -> 101
Changed lines of the file:
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@@
 	)
 	(via
-		(at 98.857 38.683)
+		(at 98.5268 38.81)
 		(size 0.4)
 		(drill 0.2)
@@
 	)
 	(via
+		(at 99.6444 37.8448)
+		(size 0.4)
+		(drill 0.2)
+		(layers "F.Cu" "B.Cu")
+		(free yes)
+		(net 2)
+	)
+	(via
 		(at 85.014 33.349)
 		(size 0.4)
@@
 	)
 	(via
-		(at 103.937 39.064)
+		(at 103.7592 39.064)
 		(size 0.4)
 		(drill 0.2)
@@
 	)
 	(segment
-		(start 100.089454 38.383154)
+		(start 99.378254 38.383154)
 		(end 100.539767 38.383154)
+		(width 0.2)
+		(layer "F.Cu")
+		(net 7)
+	)
+	(segment
+		(start 99.1416 35.839657)
+		(end 99.1416 38.1465)
+		(width 0.2)
+		(layer "F.Cu")
+		(net 7)
+	)
+	(segment
+		(start 99.1416 38.1465)
+		(end 99.378254 38.383154)
 		(width 0.2)
 		(layer "F.Cu")
@@
 	)
 	(segment
-		(start 99.1416 35.839657)
-		(end 99.1416 37.4353)
-		(width 0.2)
-		(layer "F.Cu")
-		(net 7)
-	)
-	(segment
-		(start 99.1416 37.4353)
-		(end 100.089454 38.383154)
-		(width 0.2)
-		(layer "F.Cu")
-		(net 7)
-	)
-	(segment
 		(start 100.539767 38.383154)
 		(end 102 39.843387)
@@
 	)
 	(segment
-		(start 100.332246 38.884154)
-		(end 100.023354 38.884154)
-		(width 0.2)
-		(layer "F.Cu")
-		(net 8)
-	)
-	(segment
 		(start 99.1416 33.9534)
 		(end 99.1416 31.537943)
@@
 	)
 	(segment
-		(start 98.6284 37.4892)
-		(end 98.6284 34.4666)
-		(width 0.2)
-		(layer "F.Cu")
-		(net 8)
-	)
-	(segment
-		(start 100.023354 38.884154)
-		(end 98.6284 37.4892)
-		(width 0.2)
-		(layer "F.Cu")
-		(net 8)
-	)
-	(segment
 		(start 98.6284 34.4666)
 		(end 99.1416 33.9534)
@@
 		(net 8)
 	)
+	(segment
+		(start 98.6284 38.2004)
+		(end 98.6284 34.4666)
+		(width 0.2)
+		(layer "F.Cu")
+		(net 8)
+	)
+	(segment
+		(start 99.312154 38.884154)
+		(end 98.6284 38.2004)
+		(width 0.2)
+		(layer "F.Cu")
+		(net 8)
+	)
+	(segment
+		(start 100.332246 38.884154)
+		(end 99.312154 38.884154)
+		(width 0.2)
+		(layer "F.Cu")
+		(net 8)
+	)
 	(via
 		(at 100.332246 38.884154)
@@
 	)
 	(segment
+		(start 99.7968 38.711079)
+		(end 99.7968 40.3936)
+		(width 0.2)
+		(layer "B.Cu")
+		(net 9)
+	)
+	(segment
+		(start 100.1524 34.3396)
+		(end 100.1524 38.355479)
+		(width 0.2)
+		(layer "B.Cu")
+		(net 9)
+	)
+	(segment
 		(start 99.7968 40.3936)
 		(end 100 40.5968)
@@
 	)
 	(segment
-		(start 99.7968 37.8702)
-		(end 99.7968 40.3936)
-		(width 0.2)
-		(layer "B.Cu")
-		(net 9)
-	)
-	(segment
-		(start 100.1524 37.5146)
-		(end 99.7968 37.8702)
-		(width 0.2)
-		(layer "B.Cu")
-		(net 9)
-	)
-	(segment
-		(start 100.1524 34.3396)
-		(end 100.1524 37.5146)
-		(width 0.2)
-		(layer "B.Cu")
+		(start 100.1524 38.355479)
+		(end 99.7968 38.711079)
+		(width 0.2)
+		(layer "B.Cu")
