File: PCB/SensorBoard/SensorBoard.kicad_pcb (KiCad board)
At the start: 2 copper layers, 24 x 13 mm, 13 parts, among them J1 to MAIN, Q1 2SC2712-Y, Q2 2SC2712-Y, Q3 2SC2712-Y

Commit message: ソレノイド基板作成開始
Routing:
- net GND: track 33.6 -> 35.0 mm
Changed lines of the file:
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@@
+	)
+	(segment
+		(start 52.7 35.4888)
+		(end 54.6888 33.5)
+		(width 0.3)
+		(layer "F.Cu")
+		(net 1)
 	)
 	(segment
@@
 	)
 	(segment
-		(start 52.7 40.85)
-		(end 52.7 36.3)
-		(width 0.3)
-		(layer "F.Cu")
-		(net 1)
-	)
-	(segment
-		(start 52.7 36.3)
-		(end 55.5 33.5)
-		(width 0.3)
-		(layer "F.Cu")
-		(net 1)
-	)
-	(segment
 		(start 56.800465 37.598065)
 		(end 56.800465 37.599535)
@@
 	)
 	(segment
+		(start 52.7 40.85)
+		(end 52.7 35.4888)
+		(width 0.3)
+		(layer "F.Cu")
+		(net 1)
+	)
+	(segment
+		(start 54.6888 33.5)
+		(end 55.5 33.5)
+		(width 0.3)
+		(layer "F.Cu")
+		(net 1)
+	)
+	(segment
 		(start 60.4 38.55)
 		(end 60.82 38.55)
@@
 	)
 	(segment
-		(start 54.6 36.6)
-		(end 54.6 34.4)
-		(width 0.3)
-		(layer "B.Cu")
-		(net 1)
-	)
-	(segment
 		(start 54.6 38.775)
 		(end 54.6 36.6)
@@
 	)
 	(segment
-		(start 56.726 34.726)
+		(start 54.638 33.5)
 		(end 55.5 33.5)
+		(width 0.3)
+		(layer "B.Cu")
+		(net 1)
+	)
+	(segment
+		(start 56.549 33.689)
+		(end 56.36 33.5)
+		(width 0.3)
+		(layer "B.Cu")
+		(net 1)
+	)
+	(segment
+		(start 54.5084 33.6296)
+		(end 54.638 33.5)
 		(width 0.3)
 		(layer "B.Cu")
@@
 	)
 	(segment
-		(start 54.6 34.4)
-		(end 55.5 33.5)
+		(start 56.549 34.168917)
+		(end 56.549 33.689)
 		(width 0.3)
 		(layer "B.Cu")
@@
 	)
 	(segment
+		(start 54.5084 36.5084)
+		(end 54.5084 33.6296)
+		(width 0.3)
+		(layer "B.Cu")
+		(net 1)
+	)
+	(segment
+		(start 57.106083 34.726)
+		(end 56.549 34.168917)
+		(width 0.3)
+		(layer "B.Cu")
+		(net 1)
+	)
+	(segment
 		(start 62.1 36.3)
 		(end 60.526 34.726)
@@
 	)
 	(segment
-		(start 60.526 34.726)
-		(end 56.726 34.726)
+		(start 54.6 36.6)
+		(end 54.5084 36.5084)
 		(width 0.3)
 		(layer "B.Cu")
@@
 		(layer "B.Cu")
 		(net 1)
+	)
+	(segment
+		(start 56.36 33.5)
+		(end 55.5 33.5)
+		(width 0.3)
+		(layer "B.Cu")
+		(net 1)
+	)
+	(segment
+		(start 60.526 34.726)
+		(end 57.106083 34.726)
+		(width 0.3)
+		(layer "B.Cu")
+		(net 1)
