File: PCB/SolenoidBoard/SolenoidBoard.kicad_sch (KiCad schematic)
At the start: 38 parts, among them IC1 NJW4132U2-B-TE2, J1 XT30, J2 Con_45V, J3 Con_45V, J4 Conn_01x02, J5 Con_GND, J6 Con_GND, J7 Conn_01x02, J8 Conn_01x06_Pin, J9 Conn_01x02, Q1 Q_PMOS_GSD, Q3 TPH11006NL,LQ_S, Q4 TPH11006NL,LQ_S, Q5 TPH11006NL,LQ_S, U1 TLP293, U2 TLP293, U3 TLP293, U4 TLP293

Commit message: 配線終わり
Parts:
- removed Q1: Q_PMOS_GSD, Package_TO_SOT_SMD:SOT-23-3, symbol Transistor_FET:Q_PMOS_GSD
- added Q1: Q_PMOS_GDS, Package_TO_SOT_SMD:TO-252-2, symbol Transistor_FET:Q_PMOS_GDS
- CR1: footprint SOD-323HEUS2H_TOS -> CUHS20S60:SOD-323HEUS2H_TOS
- renumbered D2 to D1, J8 to J2, J2 to J3, J3 to J4, J4 to J7, J7 to J8, Q5 to Q2, R5 to R1, R6 to R2, R7 to R3, R8 to R4, R1 to R5, R3 to R6, R2 to R7, R11 to R8
Connections:
- net +48V: now also Q1.3 (S)
- net Pch_G: now also Q1.1 (G)
- net at D1.2 (A), J3.1 (Pin_1), J4.1 (Pin_1)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: now also Q1.2 (D)

Commit message: 電圧系追加
Parts:
- added J10, J11: Conn_01x01_Pin, TestPoint:TestPoint_Loop_D2.50mm_Drill1.0mm, symbol Connector:Conn_01x01_Pin
Connections:
- net +12V: now also J10.1 (Pin_1)
- net GND: now also J11.1 (Pin_1)

Commit message: 基板外形変更
Parts:
- J1: footprint Connector_AMASS:AMASS_XT30PW-M_1x02_P2.50mm_Horizontal -> Connector_AMASS:AMASS_XT30U-M_1x02_P5.0mm_Vertical
